File: trial_project.kicad_pcb (KiCad board)
At the start: 2 copper layers, 87 x 53 mm, 14 parts, among them SW1 SW_Push, SW2 SW_Push, SW3 SW_Push, U1 MAX30102, U2 SSD1306

Commit message: completed version of project
Parts:
- moved R4 2.55 mm to (125.2, 108.0)
- moved ALARM 2.54 mm to (145.5, 108.0)
- renumbered D1 to ALARM, SW3 to DOWN, SW1 to MENU, SW2 to UP
Connections:
- U2 pad 1: +5V -> GND
- U2 pad 2: GND -> +5V
Routing:
- net GND: track 121.8 -> 48.8 mm
- net Net-(A1-A4): track 0.13 -> 59.0 mm
- net Net-(A1-A5): track 0.00 -> 57.8 mm, vias 0 -> 1
- net +5V: track 98.0 -> 129.8 mm
Other:
- board text added: "DIY SPO2"
- board text added: "U2"
Changed lines of the file:
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@@
 		(13 "F.Paste" user)
 		(15 "B.Paste" user)
-		(5 "F.SilkS" user)
-		(7 "B.SilkS" user)
+		(5 "F.SilkS" user "F.Silkscreen")
+		(7 "B.SilkS" user "B.Silkscreen")
 		(1 "F.Mask" user)
 		(3 "B.Mask" user)
 		(25 "Edge.Cuts" user)
 		(27 "Margin" user)
-		(31 "F.CrtYd" user)
-		(29 "B.CrtYd" user)
+		(31 "F.CrtYd" user "F.Courtyard")
+		(29 "B.CrtYd" user "B.Courtyard")
 		(35 "F.Fab" user)
 	)
@@
 			(plot_on_all_layers_selection 0x00000000_00000000_00000000_00000000)
 			(disableapertmacros no)
-			(usegerberextensions no)
-			(usegerberattributes yes)
-			(usegerberadvancedattributes yes)
-			(creategerberjobfile yes)
+			(usegerberextensions yes)
+			(usegerberattributes no)
+			(usegerberadvancedattributes no)
+			(creategerberjobfile no)
 			(dashed_line_dash_ratio 12.000000)
 			(dashed_line_gap_ratio 3.000000)
@@
 			(sketchdnponfab yes)
 			(crossoutdnponfab yes)
-			(subtractmaskfromsilk no)
+			(subtractmaskfromsilk yes)
 			(outputformat 1)
 			(mirror no)
-			(drillshape 1)
+			(drillshape 0)
 			(scaleselection 1)
-			(outputdirectory "")
+			(outputdirectory "gerber/")
 		)
 	)
@@
 		(at 73.66 143.51)
 		(property "Reference" "U1"
-			(at 6 9 0)
+			(at 9.34 6.49 0)
 			(unlocked yes)
 			(layer "F.SilkS")
@@
 			)
 		)
-		(fp_text user "${REFERENCE}"
-			(at -1 2.5 0)
-			(unlocked yes)
-			(layer "F.Fab")
-			(effects
-				(font
-					(size 1 1)
-					(thickness 0.15)
-				)
-			)
-		)
 		(pad "1" thru_hole rect
 			(at -5.08 -5.08)
@@
 		(descr "Generic 6mm SW tactile push button")
 		(tags "tact sw push 6mm")
-		(property "Reference" "SW2"
-			(at 3.25 -2 0)
+		(property "Reference" "UP"
+			(at 3.76 6.06 0)
 			(layer "F.SilkS")
 			(effects
@@
 		)
 		(property "Value" "SW_Push"
-			(at 3.75 6.7 0)
+			(at 2.76 -2.94 0)
 			(layer "F.Fab")
 			(effects
@@
 	(footprint "Resistor_THT:R_Axial_DIN0207_L6.3mm_D2.5mm_P7.62mm_Horizontal"
 		(layer "F.Cu")
-		(at 125.73 110.49)
+		(at 125.19 108)
 		(descr "Resistor, Axial_DIN0207 series, Axial, Horizontal, pin pitch=7.62mm, 0.25W = 1/4W, length*diameter=6.3*2.5mm^2, http://cdn-reichelt.de/documents/datenblatt/B400/1_4W%23YAG.pdf")
 		(tags "Resistor Axial_DIN0207 series Axial Horizontal pin pitch 7.62mm 0.25W = 1/4W length 6.3mm diameter 2.5mm")
@@
 		(descr "Generic 6mm SW tactile push button")
 		(tags "tact sw push 6mm")
-		(property "Reference" "SW1"
+		(property "Reference" "MENU"
 			(at 3.25 -2 0)
 			(layer "F.SilkS")
@@
 			)
 		)
-		(fp_text user "${REFERENCE}"
-			(at 0 2.5 0)
-			(unlocked yes)
-			(layer "F.Fab")
-			(effects
-				(font
-					(size 1 1)
-					(thickness 0.15)
-				)
-			)
-		)
 		(pad "1" thru_hole rect
 			(at -3.81 -10.16)
@@
 			(layers "*.Cu" "*.Mask")
 			(remove_unused_layers no)
-			(net 27 "+5V")
-			(pinfunction "VCC")
+			(net 24 "GND")
+			(pinfunction "GND")
 			(pintype "power_in")
 		)
@@
 			(layers "*.Cu" "*.Mask")
 			(remove_unused_layers no)
-			(net 24 "GND")
-			(pinfunction "GND")
+			(net 27 "+5V")
+			(pinfunction "VCC")
 			(pintype "power_in")
 		)
@@
 		(descr "Generic 6mm SW tactile push button")
 		(tags "tact sw push 6mm")
-		(property "Reference" "SW3"
-			(at 3.25 -2 0)
+		(property "Reference" "DOWN"
+			(at 3.25 6.49 0)
 			(layer "F.SilkS")
 			(effects
@@
 		)
 		(property "Value" "SW_Push"
-			(at 3.75 6.7 0)
+			(at 2.76 -2.51 0)
 			(layer "F.Fab")
 			(effects
@@
 	(footprint "LED_THT:LED_D5.0mm"
 		(layer "F.Cu")
-		(at 146.05 110.49 180)
+		(at 145.54 108 180)
 		(descr "LED, diameter 5.0mm, 2 pins, http://cdn-reichelt.de/documents/datenblatt/A500/LL-504BC2E-009.pdf, generated by kicad-footprint-generator")
 		(tags "LED")
-		(property "Reference" "D1"
+		(property "Reference" "ALARM"
 			(at 1.27 -3.96 0)
 			(layer "F.SilkS")
@@
 		(layer "Edge.Cuts")
 	)
+	(gr_text "DIY\nSPO2"
+		(at 88 148 0)
+		(layer "F.SilkS")
+		(effects
+			(font
+				(size 2 2)
+				(thickness 0.3)
+			)
+			(justify left bottom)
+		)
+	)
 	(gr_text "SDA"
 		(at 84.328 109.982 90)
@@
 		)
 	)
+	(gr_text "U2"
+		(at 96 132 0)
+		(layer "F.Fab")
+		(effects
+			(font
+				(size 1 1)
+				(thickness 0.15)
+			)
+		)
+	)
 	(segment
 		(start 119.38 110.49)
-		(end 125.73 110.49)
+		(end 122.7 110.49)
+		(width 0.127)
+		(layer "F.Cu")
+		(net 5)
+	)
+	(segment
+		(start 122.7 110.49)
+		(end 125.19 108)
 		(width 0.127)
 		(layer "F.Cu")
@@
 	)
 	(segment
+		(start 84 128.27)
+		(end 104.14 128.27)
+		(width 0.4)
+		(layer "F.Cu")
+		(net 10)
+	)
+	(segment
 		(start 83.82 106.68)
 		(end 83.82 106.812193)
@@
 	)
 	(segment
+		(start 83.82 106.68)
+		(end 83.82 128.09)
+		(width 0.4)
+		(layer "F.Cu")
+		(net 10)
+	)
+	(segment
+		(start 81.28 128.27)
+		(end 84 128.27)
+		(width 0.4)
+		(layer "F.Cu")
+		(net 10)
+	)
+	(segment
+		(start 71.12 138.43)
+		(end 81.28 128.27)
+		(width 0.4)
+		(layer "F.Cu")
+		(net 10)
+	)
+	(segment
+		(start 83.82 128.09)
+		(end 84 128.27)
+		(width 0.4)
+		(layer "F.Cu")
+		(net 10)
+	)
+	(segment
 		(start 127 121.88)
 		(end 133.31 121.88)
@@
 	)
 	(segment
-		(start 140.01 116.88)
-		(end 140.26 117.13)
-		(width 0.127)
+		(start 73.66 138.43)
+		(end 81.28 130.81)
+		(width 0.4)
 		(layer "F.Cu")
-		(net 24)
-	)
-	(segment
-		(start 146.05 116.42)
-		(end 146.76 117.13)
-		(width 0.127)
-		(layer "F.Cu")
-		(net 24)
+		(net 20)
 	)
 	(segment
-		(start 146.05 110.49)
-		(end 146.05 116.42)
-		(width 0.127)
+		(start 81.28 130.81)
+		(end 104.14 130.81)
+		(width 0.4)
 		(layer "F.Cu")
-		(net 24)
+		(net 20)
 	)
-	(segment
-		(start 140.26 133.06)
-		(end 146.76 133.06)
-		(width 0.127)
-		(layer "F.Cu")
-		(net 24)
+	(via
+		(at 81.28 130.81)
+		(size 0.6)
+		(drill 0.3)
+		(layers "F.Cu" "B.Cu")
+		(net 20)
 	)
 	(segment
-		(start 146.76 144.49)
-		(end 140.26 144.49)
-		(width 0.127)
-		(layer "F.Cu")
-		(net 24)
+		(start 81.28 106.68)
+		(end 81.28 130.81)
+		(width 0.4)
+		(layer "B.Cu")
+		(net 20)
 	)
 	(segment
-		(start 129.325001 135.635001)
-		(end 127 133.31)
+		(start 140.01 116.88)
+		(end 140.26 117.13)
 		(width 0.127)
 		(layer "F.Cu")
@@
 	)
 	(segment
-		(start 140.26 133.06)
-		(end 137.684999 135.635001)
+		(start 146.05 116.42)
+		(end 146.76 117.13)
 		(width 0.127)
 		(layer "F.Cu")
@@
 	)
 	(segment
-		(start 137.684999 135.635001)
-		(end 129.325001 135.635001)
-		(width 0.127)
-		(layer "F.Cu")
-		(net 24)
-	)
-	(segment
-		(start 146.76 133.06)
-		(end 148 134.3)
-		(width 0.127)
-		(layer "F.Cu")
-		(net 24)
-	)
-	(segment
 		(start 140.26 117.13)
 		(end 146.76 117.13)
@@
 	)
 	(segment
-		(start 148 143.25)
-		(end 146.76 144.49)
-		(width 0.127)
-		(layer "F.Cu")
-		(net 24)
-	)
-	(segment
 		(start 120.69 138.43)
 		(end 127 144.74)
@@
 	)
 	(segment
-		(start 148 134.3)
-		(end 148 143.25)
-		(width 0.127)
-		(layer "F.Cu")
-		(net 24)
-	)
-	(segment
 		(start 139 131.8)
 		(end 140.26 133.06)
@@
 	)
 	(segment
-		(start 114.3 143.51)
-		(end 119.38 138.43)
-		(width 0.127)
-		(layer "B.Cu")
-		(net 24)
-	)
-	(segment
 		(start 140.26 117.13)
 		(end 139 118.39)
@@
 	)
 	(segment
-		(start 119.38 138.43)
-		(end 121.88 138.43)
-		(width 0.127)
-		(layer "B.Cu")
-		(net 24)
-	)
-	(segment
-		(start 104.14 143.51)
-		(end 114.3 143.51)
-		(width 0.127)
-		(layer "B.Cu")
-		(net 24)
-	)
-	(segment
-		(start 121.88 138.43)
-		(end 127 133.31)
-		(width 0.127)
+		(start 76.2 138.43)
+		(end 76.2 139.2)
+		(width 0.4)
 		(layer "B.Cu")
 		(net 24)
 	)
 	(segment
-		(start 78.74 138.43)
-		(end 104.14 138.43)
+		(start 118 152)
+		(end 132 152)
 		(width 0.127)
 		(layer "F.Cu")
@@
 	)
 	(segment
-		(start 118 152)
-		(end 132 152)
-		(width 0.127)
+		(start 78.74 138.43)
+		(end 104.14 138.43)
+		(width 0.4)
 		(layer "F.Cu")
 		(net 27)
@@
 	)
 	(segment
-		(start 133.35 110.49)
-		(end 143.51 110.49)
+		(start 78.74 106.68)
+		(end 78.74 138.43)
+		(width 0.4)
+		(layer "B.Cu")
+		(net 27)
+	)
+	(segment
+		(start 132.81 108)
+		(end 143 108)
 		(width 0.127)
 		(layer "F.Cu")
@@
 		(min_thickness 0.25)
 		(filled_areas_thickness no)
-		(fill
+		(fill yes
 			(thermal_gap 0.5)
 			(thermal_bridge_width 0.5)
