File: trial_project.kicad_sch (KiCad schematic)
At the start: 14 parts, among them SW1 SW_Push, SW2 SW_Push, SW3 SW_Push, U1 MAX30102, U2 SSD1306

Commit message: PCB design is ongoing
an issue with track between VCC and GND
Changed lines of the file:
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@@
 	(wire
 		(pts
-			(xy 193.04 100.33) (xy 193.04 105.41)
+			(xy 193.04 100.33) (xy 193.04 114.3)
 		)
 		(stroke
@@
 	(symbol
 		(lib_id "power:GND")
-		(at 193.04 105.41 0)
+		(at 193.04 114.3 0)
 		(unit 1)
 		(exclude_from_sim no)
@@
 		(fields_autoplaced yes)
 		(property "Reference" "#PWR011"
-			(at 193.04 111.76 0)
+			(at 193.04 120.65 0)
 			(effects
 				(font
@@
 		)
 		(property "Value" "GND"
-			(at 193.04 110.49 0)
+			(at 193.04 119.38 0)
 			(effects
 				(font
@@
 		)
 		(property "Footprint" ""
-			(at 193.04 105.41 0)
+			(at 193.04 114.3 0)
 			(effects
 				(font
@@
 		)
 		(property "Datasheet" ""
-			(at 193.04 105.41 0)
+			(at 193.04 114.3 0)
 			(effects
 				(font
@@
 		)
 		(property "Description" "Power symbol creates a global label with name \"GND\" , ground"
-			(at 193.04 105.41 0)
-			(effects
-				(font
+			(at 193.04 114.3 0)
+			(effects
+				(font

Commit message: completed version of project
Connections:
- net +5V: now also U2.2 (VCC); no longer U2.1 (VCC)
- net GND: now also U2.1 (GND); no longer U2.2 (GND)
